Commit message: Updated the p3bot model

File: rtb-data/rtbdata/xacro/p3bot_description/urdf/P3Bot_scaled.urdf (robot description, URDF)
Before this commit: robot P3Bot_description, 21 links, 20 joints
Joints:
- joint base_link2low_body: origin xyz=0 0 0.21 rpy=0 0 0 -> xyz=0 0 0.21 rpy=0 0 -1.57

Commit message: Added the second arm

File: rtb-data/rtbdata/xacro/p3bot_description/urdf/P3Bot_scaled.urdf (robot description, URDF)
Before this commit: robot P3Bot_description, 21 links, 20 joints
Links:
- added link left_arm, mass 1.697; collision mesh filename=meshes/arm_base_link.STL; visual mesh filename=meshes/arm_base_link.STL
- added link left_arm_bracelet_link, mass 0.5; collision mesh filename=meshes/bracelet_with_vision_link.STL; visual mesh filename=meshes/bracelet_with_vision_link.STL
- added link left_arm_camera_color_frame
- added link left_arm_camera_depth_frame
- added link left_arm_camera_link
- added link left_arm_end_effector_link
- added link left_arm_forearm_link, mass 0.9302; collision mesh filename=meshes/forearm_link.STL; visual mesh filename=meshes/forearm_link.STL
- added link left_arm_half_arm_1_link, mass 1.1636; collision mesh filename=meshes/half_arm_1_link.STL; visual mesh filename=meshes/half_arm_1_link.STL
- added link left_arm_half_arm_2_link, mass 1.1636; collision mesh filename=meshes/half_arm_2_link.STL; visual mesh filename=meshes/half_arm_2_link.STL
- added link left_arm_shoulder_link, mass 1.3773; collision mesh filename=meshes/shoulder_link.STL; visual mesh filename=meshes/shoulder_link.STL
- added link left_arm_spherical_wrist_1_link, mass 0.6781; collision mesh filename=meshes/spherical_wrist_1_link.STL; visual mesh filename=meshes/spherical_wrist_1_link.STL
- added link left_arm_spherical_wrist_2_link, mass 0.6781; collision mesh filename=meshes/spherical_wrist_2_link.STL; visual mesh filename=meshes/spherical_wrist_2_link.STL
- added link left_arm_tool_frame
Joints:
- added joint chess2left_arm: type fixed, parent chess, child left_arm, origin xyz=-0.053182 0.066416 0.34067 rpy=-2.0071 0 1.5708, axis 0 0 0
- added joint left_arm_camera_module: type fixed, parent left_arm_end_effector_link, child left_arm_camera_link, origin xyz=0 0.05639 -0.00305 rpy=3.14159265358979 3.14159265358979 0
- added joint left_arm_color_module: type fixed, parent left_arm_end_effector_link, child left_arm_camera_color_frame, origin xyz=0 0.05639 -0.00305 rpy=3.14159265358979 3.14159265358979 0
- added joint left_arm_depth_module: type fixed, parent left_arm_end_effector_link, child left_arm_camera_depth_frame, origin xyz=0.0275 0.066 -0.00305 rpy=3.14159265358979 3.14159265358979 0
- added joint left_arm_end_effector: type fixed, parent left_arm_bracelet_link, child left_arm_end_effector_link, origin xyz=0 0 -0.0615250000000001 rpy=3.14159265358979 1.09937075168372E-32 0, axis 0 0 0
- added joint left_arm_joint_1: type continuous, parent left_arm, child left_arm_shoulder_link, origin xyz=0 0 0.15643 rpy=3.1416 2.7629E-18 -4.9305E-36, axis 0 0 1, limit effort=39 velocity=1.3963
- added joint left_arm_joint_2: type revolute, parent left_arm_shoulder_link, child left_arm_half_arm_1_link, origin xyz=0 0.005375 -0.12838 rpy=1.5708 2.1343E-17 -1.1102E-16, axis 0 0 1, limit lower=-2.24 upper=2.24 effort=39 velocity=1.3963
- added joint left_arm_joint_3: type continuous, parent left_arm_half_arm_1_link, child left_arm_half_arm_2_link, origin xyz=0 -0.21038 -0.006375 rpy=-1.5708 1.2326E-32 -2.9122E-16, axis 0 0 1, limit effort=39 velocity=1.3963
- added joint left_arm_joint_4: type revolute, parent left_arm_half_arm_2_link, child left_arm_forearm_link, origin xyz=0 0.006375 -0.21038 rpy=1.5708 -6.6954E-17 -1.6653E-16, axis 0 0 1, limit lower=-2.57 upper=2.57 effort=39 velocity=1.3963
- added joint left_arm_joint_5: type continuous, parent left_arm_forearm_link, child left_arm_spherical_wrist_1_link, origin xyz=0 -0.20843 -0.006375 rpy=-1.5708 2.2204E-16 -6.373E-17, axis 0 0 1, limit effort=9 velocity=1.2218
- added joint left_arm_joint_6: type revolute, parent left_arm_spherical_wrist_1_link, child left_arm_spherical_wrist_2_link, origin xyz=0 0.00017505 -0.10593 rpy=1.5708 9.2076E-28 -8.2157E-15, axis 0 0 1, limit lower=-2.09 upper=2.09 effort=9 velocity=1.2218
- added joint left_arm_joint_7: type continuous, parent left_arm_spherical_wrist_2_link, child left_arm_bracelet_link, origin xyz=0 -0.10593 -0.00017505 rpy=-1.5708 -5.5511E-17 9.6396E-17, axis 0 0 1, limit effort=9 velocity=1.2218
- added joint left_arm_tool_frame_joint: type fixed, parent left_arm_end_effector_link, child left_arm_tool_frame, origin xyz=0 0 0.120 rpy=0 0 0, axis 0 0 0

Commit message: Updated the p3bot urdf

File: rtb-data/rtbdata/xacro/p3bot_description/urdf/P3Bot_scaled.urdf (robot description, URDF)
Before this commit: robot P3Bot_description, 34 links, 33 joints
Links:
- link left_arm: geometry collision mesh filename=p3bot_description/meshes/arm_base_link.STL; visual mesh filename=p3bot_description/meshes/arm_base_link.STL
- link left_arm_bracelet_link: geometry collision mesh filename=p3bot_description/meshes/bracelet_with_vision_link.STL; visual mesh filename=p3bot_description/meshes/bracelet_with_vision_link.STL
- link left_arm_forearm_link: geometry collision mesh filename=p3bot_description/meshes/forearm_link.STL; visual mesh filename=p3bot_description/meshes/forearm_link.STL
- link left_arm_half_arm_1_link: geometry collision mesh filename=p3bot_description/meshes/half_arm_1_link.STL; visual mesh filename=p3bot_description/meshes/half_arm_1_link.STL
- link left_arm_half_arm_2_link: geometry collision mesh filename=p3bot_description/meshes/half_arm_2_link.STL; visual mesh filename=p3bot_description/meshes/half_arm_2_link.STL
- link left_arm_shoulder_link: geometry collision mesh filename=p3bot_description/meshes/shoulder_link.STL; visual mesh filename=p3bot_description/meshes/shoulder_link.STL
- link left_arm_spherical_wrist_1_link: geometry collision mesh filename=p3bot_description/meshes/spherical_wrist_1_link.STL; visual mesh filename=p3bot_description/meshes/spherical_wrist_1_link.STL
- link left_arm_spherical_wrist_2_link: geometry collision mesh filename=p3bot_description/meshes/spherical_wrist_2_link.STL; visual mesh filename=p3bot_description/meshes/spherical_wrist_2_link.STL

Commit message: Trying to do stable the P3Bot two arm

File: rtb-data/rtbdata/xacro/p3bot_description/urdf/P3Bot_scaled.urdf (robot description, URDF)
Before this commit: robot P3Bot_description, 34 links, 33 joints
Links:
- added link left_arm_left_inner_finger, mass 0.0104003125914103; collision mesh filename=meshes/collision/robotiq_arg2f_85_inner_finger.dae scale=0.001 0.001 0.001; visual mesh filename=meshes/visual/robotiq_arg2f_85_inner_finger.dae scale=0.001 0.001 0.001
- added link left_arm_left_inner_finger_pad; collision box size=0.022 0.00635 0.0375; visual box size=0.022 0.00635 0.0375
- added link left_arm_left_inner_knuckle, mass 0.0271177346495152; collision mesh filename=meshes/collision/robotiq_arg2f_85_inner_knuckle.dae scale=0.001 0.001 0.001; visual mesh filename=meshes/visual/robotiq_arg2f_85_inner_knuckle.dae scale=0.001 0.001 0.001
- added link left_arm_left_outer_finger, mass 0.022614240507152; collision mesh filename=meshes/collision/robotiq_arg2f_85_outer_finger.dae scale=0.001 0.001 0.001; visual mesh filename=meshes/visual/robotiq_arg2f_85_outer_finger.dae scale=0.001 0.001 0.001
- added link left_arm_left_outer_knuckle, mass 0.00853198276973456; collision mesh filename=meshes/collision/robotiq_arg2f_85_outer_knuckle.dae scale=0.001 0.001 0.001; visual mesh filename=meshes/visual/robotiq_arg2f_85_outer_knuckle.dae scale=0.001 0.001 0.001
- added link left_arm_right_inner_finger, mass 0.0104003125914103; collision mesh filename=meshes/collision/robotiq_arg2f_85_inner_finger.dae scale=0.001 0.001 0.001; visual mesh filename=meshes/visual/robotiq_arg2f_85_inner_finger.dae scale=0.001 0.001 0.001
- added link left_arm_right_inner_finger_pad; collision box size=0.022 0.00635 0.0375; visual box size=0.022 0.00635 0.0375
- added link left_arm_right_inner_knuckle, mass 0.0271177346495152; collision mesh filename=/meshes/collision/robotiq_arg2f_85_inner_knuckle.dae scale=0.001 0.001 0.001; visual mesh filename=meshes/visual/robotiq_arg2f_85_inner_knuckle.dae scale=0.001 0.001 0.001
- added link left_arm_right_outer_finger, mass 0.022614240507152; collision mesh filename=meshes/collision/robotiq_arg2f_85_outer_finger.dae scale=0.001 0.001 0.001; visual mesh filename=meshes/visual/robotiq_arg2f_85_outer_finger.dae scale=0.001 0.001 0.001
- added link left_arm_right_outer_knuckle, mass 0.00853198276973456; collision mesh filename=meshes/collision/robotiq_arg2f_85_outer_knuckle.dae scale=0.001 0.001 0.001; visual mesh filename=meshes/visual/robotiq_arg2f_85_outer_knuckle.dae scale=0.001 0.001 0.001
- added link left_arm_robotiq_arg2f_base_link, mass 0.22652; collision mesh filename=meshes/collision/robotiq_arg2f_base_link_85.stl; visual mesh filename=meshes/collision/robotiq_arg2f_base_link_85.stl
- added link right_arm_left_inner_finger, mass 0.0104003125914103; collision mesh filename=meshes/collision/robotiq_arg2f_85_inner_finger.dae scale=0.001 0.001 0.001; visual mesh filename=meshes/visual/robotiq_arg2f_85_inner_finger.dae scale=0.001 0.001 0.001
- added link right_arm_left_inner_finger_pad; collision box size=0.022 0.00635 0.0375; visual box size=0.022 0.00635 0.0375
- added link right_arm_left_inner_knuckle, mass 0.0271177346495152; collision mesh filename=meshes/collision/robotiq_arg2f_85_inner_knuckle.dae scale=0.001 0.001 0.001; visual mesh filename=meshes/visual/robotiq_arg2f_85_inner_knuckle.dae scale=0.001 0.001 0.001
- added link right_arm_left_outer_finger, mass 0.022614240507152; collision mesh filename=meshes/collision/robotiq_arg2f_85_outer_finger.dae scale=0.001 0.001 0.001; visual mesh filename=meshes/visual/robotiq_arg2f_85_outer_finger.dae scale=0.001 0.001 0.001
- added link right_arm_left_outer_knuckle, mass 0.00853198276973456; collision mesh filename=meshes/collision/robotiq_arg2f_85_outer_knuckle.dae scale=0.001 0.001 0.001; visual mesh filename=meshes/visual/robotiq_arg2f_85_outer_knuckle.dae scale=0.001 0.001 0.001
- added link right_arm_right_inner_finger, mass 0.0104003125914103; collision mesh filename=meshes/collision/robotiq_arg2f_85_inner_finger.dae scale=0.001 0.001 0.001; visual mesh filename=meshes/visual/robotiq_arg2f_85_inner_finger.dae scale=0.001 0.001 0.001
- added link right_arm_right_inner_finger_pad; collision box size=0.022 0.00635 0.0375; visual box size=0.022 0.00635 0.0375
- added link right_arm_right_inner_knuckle, mass 0.0271177346495152; collision mesh filename=/meshes/collision/robotiq_arg2f_85_inner_knuckle.dae scale=0.001 0.001 0.001; visual mesh filename=meshes/visual/robotiq_arg2f_85_inner_knuckle.dae scale=0.001 0.001 0.001
- added link right_arm_right_outer_finger, mass 0.022614240507152; collision mesh filename=meshes/collision/robotiq_arg2f_85_outer_finger.dae scale=0.001 0.001 0.001; visual mesh filename=meshes/visual/robotiq_arg2f_85_outer_finger.dae scale=0.001 0.001 0.001
- added link right_arm_right_outer_knuckle, mass 0.00853198276973456; collision mesh filename=meshes/collision/robotiq_arg2f_85_outer_knuckle.dae scale=0.001 0.001 0.001; visual mesh filename=meshes/visual/robotiq_arg2f_85_outer_knuckle.dae scale=0.001 0.001 0.001
- added link right_arm_robotiq_arg2f_base_link, mass 0.22652; collision mesh filename=meshes/collision/robotiq_arg2f_base_link_85.stl; visual mesh filename=meshes/collision/robotiq_arg2f_base_link_85.stl
Joints:
- added joint left_arm_finger_joint: type revolute, parent left_arm_robotiq_arg2f_base_link, child left_arm_left_outer_knuckle, origin xyz=0 -0.0306011 0.054904 rpy=0 0 3.141592653589793, axis 1 0 0, limit lower=0 upper=0.8 effort=1000 velocity=2.0
- added joint left_arm_gripper_base_joint: type fixed, parent left_arm_end_effector_link, child left_arm_robotiq_arg2f_base_link, origin xyz=0.0 0.0 0.0 rpy=0.0 0.0 1.57
- added joint left_arm_left_inner_finger_joint: type revolute, parent left_arm_left_outer_finger, child left_arm_left_inner_finger, origin xyz=0 0.0061 0.0471 rpy=0 0 0, axis 1 0 0, limit lower=-0.8757 upper=0.8757 effort=1000 velocity=2.0, mimic joint=left_arm_finger_joint multiplier=-1 offset=0
- added joint left_arm_left_inner_finger_pad_joint: type fixed, parent left_arm_left_inner_finger, child left_arm_left_inner_finger_pad, origin xyz=0 -0.0220203446692936 0.03242 rpy=0 0 0, axis 0 0 1
- added joint left_arm_left_inner_knuckle_joint: type revolute, parent left_arm_robotiq_arg2f_base_link, child left_arm_left_inner_knuckle, origin xyz=0 -0.0127 0.06142 rpy=0 0 3.141592653589793, axis 1 0 0, limit lower=0 upper=0.8757 effort=1000 velocity=2.0, mimic joint=left_arm_finger_joint multiplier=1 offset=0
- added joint left_arm_left_outer_finger_joint: type fixed, parent left_arm_left_outer_knuckle, child left_arm_left_outer_finger, origin xyz=0 0.0315 -0.0041 rpy=0 0 0, axis 1 0 0
- added joint left_arm_right_inner_finger_joint: type revolute, parent left_arm_right_outer_finger, child left_arm_right_inner_finger, origin xyz=0 0.0061 0.0471 rpy=0 0 0, axis 1 0 0, limit lower=-0.8757 upper=0.8757 effort=1000 velocity=2.0, mimic joint=left_arm_finger_joint multiplier=-1 offset=0
- added joint left_arm_right_inner_finger_pad_joint: type fixed, parent left_arm_right_inner_finger, child left_arm_right_inner_finger_pad, origin xyz=0 -0.0220203446692936 0.03242 rpy=0 0 0, axis 0 0 1
- added joint left_arm_right_inner_knuckle_joint: type revolute, parent left_arm_robotiq_arg2f_base_link, child left_arm_right_inner_knuckle, origin xyz=0 0.0127 0.06142 rpy=0 0 0.0, axis 1 0 0, limit lower=0 upper=0.8757 effort=1000 velocity=2.0, mimic joint=left_arm_finger_joint multiplier=1 offset=0
- added joint left_arm_right_outer_finger_joint: type fixed, parent left_arm_right_outer_knuckle, child left_arm_right_outer_finger, origin xyz=0 0.0315 -0.0041 rpy=0 0 0, axis 1 0 0
- added joint left_arm_right_outer_knuckle_joint: type revolute, parent left_arm_robotiq_arg2f_base_link, child left_arm_right_outer_knuckle, origin xyz=0 0.0306011 0.054904 rpy=0 0 0, axis 1 0 0, limit lower=0 upper=0.81 effort=1000 velocity=2.0, mimic joint=left_arm_finger_joint multiplier=1 offset=0
- added joint right_arm_finger_joint: type revolute, parent right_arm_robotiq_arg2f_base_link, child right_arm_left_outer_knuckle, origin xyz=0 -0.0306011 0.054904 rpy=0 0 3.141592653589793, axis 1 0 0, limit lower=0 upper=0.8 effort=1000 velocity=2.0
- added joint right_arm_gripper_base_joint: type fixed, parent right_arm_end_effector_link, child right_arm_robotiq_arg2f_base_link, origin xyz=0.0 0.0 0.0 rpy=0.0 0.0 1.57
- added joint right_arm_left_inner_finger_joint: type revolute, parent right_arm_left_outer_finger, child right_arm_left_inner_finger, origin xyz=0 0.0061 0.0471 rpy=0 0 0, axis 1 0 0, limit lower=-0.8757 upper=0.8757 effort=1000 velocity=2.0, mimic joint=right_arm_finger_joint multiplier=-1 offset=0
- added joint right_arm_left_inner_finger_pad_joint: type fixed, parent right_arm_left_inner_finger, child right_arm_left_inner_finger_pad, origin xyz=0 -0.0220203446692936 0.03242 rpy=0 0 0, axis 0 0 1
- added joint right_arm_left_inner_knuckle_joint: type revolute, parent right_arm_robotiq_arg2f_base_link, child right_arm_left_inner_knuckle, origin xyz=0 -0.0127 0.06142 rpy=0 0 3.141592653589793, axis 1 0 0, limit lower=0 upper=0.8757 effort=1000 velocity=2.0, mimic joint=right_arm_finger_joint multiplier=1 offset=0
- added joint right_arm_left_outer_finger_joint: type fixed, parent right_arm_left_outer_knuckle, child right_arm_left_outer_finger, origin xyz=0 0.0315 -0.0041 rpy=0 0 0, axis 1 0 0
- added joint right_arm_right_inner_finger_joint: type revolute, parent right_arm_right_outer_finger, child right_arm_right_inner_finger, origin xyz=0 0.0061 0.0471 rpy=0 0 0, axis 1 0 0, limit lower=-0.8757 upper=0.8757 effort=1000 velocity=2.0, mimic joint=right_arm_finger_joint multiplier=-1 offset=0
- added joint right_arm_right_inner_finger_pad_joint: type fixed, parent right_arm_right_inner_finger, child right_arm_right_inner_finger_pad, origin xyz=0 -0.0220203446692936 0.03242 rpy=0 0 0, axis 0 0 1
- added joint right_arm_right_inner_knuckle_joint: type revolute, parent right_arm_robotiq_arg2f_base_link, child right_arm_right_inner_knuckle, origin xyz=0 0.0127 0.06142 rpy=0 0 0.0, axis 1 0 0, limit lower=0 upper=0.8757 effort=1000 velocity=2.0, mimic joint=right_arm_finger_joint multiplier=1 offset=0
- added joint right_arm_right_outer_finger_joint: type fixed, parent right_arm_right_outer_knuckle, child right_arm_right_outer_finger, origin xyz=0 0.0315 -0.0041 rpy=0 0 0, axis 1 0 0
- added joint right_arm_right_outer_knuckle_joint: type revolute, parent right_arm_robotiq_arg2f_base_link, child right_arm_right_outer_knuckle, origin xyz=0 0.0306011 0.054904 rpy=0 0 0, axis 1 0 0, limit lower=0 upper=0.81 effort=1000 velocity=2.0, mimic joint=right_arm_finger_joint multiplier=1 offset=0

Commit message: Fixed the P3Bot urdf

File: rtb-data/rtbdata/xacro/p3bot_description/urdf/P3Bot_scaled.urdf (robot description, URDF)
Before this commit: robot P3Bot_description, 56 links, 55 joints
Links:
- removed link left_arm_left_inner_finger
- removed link left_arm_left_inner_finger_pad
- removed link left_arm_left_inner_knuckle
- removed link left_arm_left_outer_finger
- removed link left_arm_left_outer_knuckle
- removed link left_arm_right_inner_finger
- removed link left_arm_right_inner_finger_pad
- removed link left_arm_right_inner_knuckle
- removed link left_arm_right_outer_finger
- removed link left_arm_right_outer_knuckle
- removed link left_arm_robotiq_arg2f_base_link
- removed link right_arm_left_inner_finger
- removed link right_arm_left_inner_finger_pad
- removed link right_arm_left_inner_knuckle
- removed link right_arm_left_outer_finger
- removed link right_arm_left_outer_knuckle
- removed link right_arm_right_inner_finger
- removed link right_arm_right_inner_finger_pad
- removed link right_arm_right_inner_knuckle
- removed link right_arm_right_outer_finger
- removed link right_arm_right_outer_knuckle
- removed link right_arm_robotiq_arg2f_base_link
Joints:
- removed joint left_arm_finger_joint
- removed joint left_arm_gripper_base_joint
- removed joint left_arm_left_inner_finger_joint
- removed joint left_arm_left_inner_finger_pad_joint
- removed joint left_arm_left_inner_knuckle_joint
- removed joint left_arm_left_outer_finger_joint
- removed joint left_arm_right_inner_finger_joint
- removed joint left_arm_right_inner_finger_pad_joint
- removed joint left_arm_right_inner_knuckle_joint
- removed joint left_arm_right_outer_finger_joint
- removed joint left_arm_right_outer_knuckle_joint
- removed joint right_arm_finger_joint
- removed joint right_arm_gripper_base_joint
- removed joint right_arm_left_inner_finger_joint
- removed joint right_arm_left_inner_finger_pad_joint
- removed joint right_arm_left_inner_knuckle_joint
- removed joint right_arm_left_outer_finger_joint
- removed joint right_arm_right_inner_finger_joint
- removed joint right_arm_right_inner_finger_pad_joint
- removed joint right_arm_right_inner_knuckle_joint
- removed joint right_arm_right_outer_finger_joint
- removed joint right_arm_right_outer_knuckle_joint
