Commit message: added the grippers

File: rtb-data/rtbdata/xacro/p3bot_description/urdf/P3Bot_scaled.urdf (robot description, URDF)
Before this commit: robot P3Bot_description, 34 links, 33 joints
Links:
- added link left_arm_left_inner_finger, mass 0.0104003125914103; collision mesh filename=p3bot_description/meshes/collision/robotiq_arg2f_85_inner_f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 scale=0.001 0.001 0.001; visual mesh filename=p3bot_description/meshes/visual/robotiq_arg2f_85_inner_fing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 scale=0.001 0.001 0.001
- added link left_arm_left_inner_finger_pad; collision box size=0.022 0.00635 0.0375; visual box size=0.022 0.00635 0.0375
- added link left_arm_left_inner_knuckle, mass 0.0271177346495152; collision mesh filename=p3bot_description/meshes/collision/robotiq_arg2f_85_inner_k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 scale=0.001 0.001 0.001; visual mesh filename=p3bot_description/meshes/visual/robotiq_arg2f_85_inner_knuc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 scale=0.001 0.001 0.001
- added link left_arm_left_outer_finger, mass 0.022614240507152; collision mesh filename=p3bot_description/meshes/collision/robotiq_arg2f_85_outer_f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 scale=0.001 0.001 0.001; visual mesh filename=p3bot_description/meshes/visual/robotiq_arg2f_85_outer_fing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 scale=0.001 0.001 0.001
- added link left_arm_left_outer_knuckle, mass 0.00853198276973456; collision mesh filename=p3bot_description/meshes/collision/robotiq_arg2f_85_outer_k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 scale=0.001 0.001 0.001; visual mesh filename=p3bot_description/meshes/visual/robotiq_arg2f_85_outer_knuc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 scale=0.001 0.001 0.001
- added link left_arm_right_inner_finger, mass 0.0104003125914103; collision mesh filename=p3bot_description/meshes/collision/robotiq_arg2f_85_inner_f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 scale=0.001 0.001 0.001; visual mesh filename=p3bot_description/meshes/visual/robotiq_arg2f_85_inner_fing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 scale=0.001 0.001 0.001
- added link left_arm_right_inner_finger_pad; collision box size=0.022 0.00635 0.0375; visual box size=0.022 0.00635 0.0375
- added link left_arm_right_inner_knuckle, mass 0.0271177346495152; collision mesh filename=p3bot_description/meshes/collision/robotiq_arg2f_85_inner_k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 scale=0.001 0.001 0.001; visual mesh filename=p3bot_description/meshes/visual/robotiq_arg2f_85_inner_knuc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 scale=0.001 0.001 0.001
- added link left_arm_right_outer_finger, mass 0.022614240507152; collision mesh filename=p3bot_description/meshes/collision/robotiq_arg2f_85_outer_f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 scale=0.001 0.001 0.001; visual mesh filename=p3bot_description/meshes/visual/robotiq_arg2f_85_outer_fing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 scale=0.001 0.001 0.001
- added link left_arm_right_outer_knuckle, mass 0.00853198276973456; collision mesh filename=p3bot_description/meshes/collision/robotiq_arg2f_85_outer_k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 scale=0.001 0.001 0.001; visual mesh filename=p3bot_description/meshes/visual/robotiq_arg2f_85_outer_knuc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 scale=0.001 0.001 0.001
- added link left_arm_robotiq_arg2f_base_link, mass 0.22652; collision mesh filename=p3bot_description/meshes/collision/robotiq_arg2f_base_link_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; visual mesh filename=p3bot_description/meshes/collision/robotiq_arg2f_base_link_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
- added link right_arm_left_inner_finger, mass 0.0104003125914103; collision mesh filename=p3bot_description/meshes/collision/robotiq_arg2f_85_inner_f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 scale=0.001 0.001 0.001; visual mesh filename=p3bot_description/meshes/visual/robotiq_arg2f_85_inner_fing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 scale=0.001 0.001 0.001
- added link right_arm_left_inner_finger_pad; collision box size=0.022 0.00635 0.0375; visual box size=0.022 0.00635 0.0375
- added link right_arm_left_inner_knuckle, mass 0.0271177346495152; collision mesh filename=p3bot_description/meshes/collision/robotiq_arg2f_85_inner_k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 scale=0.001 0.001 0.001; visual mesh filename=p3bot_description/meshes/visual/robotiq_arg2f_85_inner_knuc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 scale=0.001 0.001 0.001
- added link right_arm_left_outer_finger, mass 0.022614240507152; collision mesh filename=p3bot_description/meshes/collision/robotiq_arg2f_85_outer_f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 scale=0.001 0.001 0.001; visual mesh filename=p3bot_description/meshes/visual/robotiq_arg2f_85_outer_fing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 scale=0.001 0.001 0.001
- added link right_arm_left_outer_knuckle, mass 0.00853198276973456; collision mesh filename=p3bot_description/meshes/collision/robotiq_arg2f_85_outer_k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 scale=0.001 0.001 0.001; visual mesh filename=p3bot_description/meshes/visual/robotiq_arg2f_85_outer_knuc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 scale=0.001 0.001 0.001
- added link right_arm_right_inner_finger, mass 0.0104003125914103; collision mesh filename=p3bot_description/meshes/collision/robotiq_arg2f_85_inner_f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 scale=0.001 0.001 0.001; visual mesh filename=p3bot_description/meshes/visual/robotiq_arg2f_85_inner_fing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 scale=0.001 0.001 0.001
- added link right_arm_right_inner_finger_pad; collision box size=0.022 0.00635 0.0375; visual box size=0.022 0.00635 0.0375
- added link right_arm_right_inner_knuckle, mass 0.0271177346495152; collision mesh filename=p3bot_description/meshes/collision/robotiq_arg2f_85_inner_k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 scale=0.001 0.001 0.001; visual mesh filename=p3bot_description/meshes/visual/robotiq_arg2f_85_inner_knuc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 scale=0.001 0.001 0.001
- added link right_arm_right_outer_finger, mass 0.022614240507152; collision mesh filename=p3bot_description/meshes/collision/robotiq_arg2f_85_outer_f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 scale=0.001 0.001 0.001; visual mesh filename=p3bot_description/meshes/visual/robotiq_arg2f_85_outer_fing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 scale=0.001 0.001 0.001
- added link right_arm_right_outer_knuckle, mass 0.00853198276973456; collision mesh filename=p3bot_description/meshes/collision/robotiq_arg2f_85_outer_k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 scale=0.001 0.001 0.001; visual mesh filename=p3bot_description/meshes/visual/robotiq_arg2f_85_outer_knuc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 scale=0.001 0.001 0.001
- added link right_arm_robotiq_arg2f_base_link, mass 0.22652; collision mesh filename=p3bot_description/meshes/collision/robotiq_arg2f_base_link_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; visual mesh filename=p3bot_description/meshes/collision/robotiq_arg2f_base_link_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
Joints:
- added joint left_arm_finger_joint: type revolute, parent left_arm_robotiq_arg2f_base_link, child left_arm_left_outer_knuckle, origin xyz=0 -0.0306011 0.054904 rpy=0 0 3.141592653589793, axis 1 0 0, limit lower=0 upper=0.8 effort=1000 velocity=2.0
- added joint left_arm_gripper_base_joint: type fixed, parent left_arm_end_effector_link, child left_arm_robotiq_arg2f_base_link, origin xyz=0.0 0.0 0.0 rpy=0.0 0.0 1.57
- added joint left_arm_left_inner_finger_joint: type revolute, parent left_arm_left_outer_finger, child left_arm_left_inner_finger, origin xyz=0 0.0061 0.0471 rpy=0 0 0, axis 1 0 0, limit lower=-0.8757 upper=0.8757 effort=1000 velocity=2.0, mimic joint=left_arm_finger_joint multiplier=-1 offset=0
- added joint left_arm_left_inner_finger_pad_joint: type fixed, parent left_arm_left_inner_finger, child left_arm_left_inner_finger_pad, origin xyz=0 -0.0220203446692936 0.03242 rpy=0 0 0, axis 0 0 1
- added joint left_arm_left_inner_knuckle_joint: type revolute, parent left_arm_robotiq_arg2f_base_link, child left_arm_left_inner_knuckle, origin xyz=0 -0.0127 0.06142 rpy=0 0 3.141592653589793, axis 1 0 0, limit lower=0 upper=0.8757 effort=1000 velocity=2.0, mimic joint=left_arm_finger_joint multiplier=1 offset=0
- added joint left_arm_left_outer_finger_joint: type fixed, parent left_arm_left_outer_knuckle, child left_arm_left_outer_finger, origin xyz=0 0.0315 -0.0041 rpy=0 0 0, axis 1 0 0
- added joint left_arm_right_inner_finger_joint: type revolute, parent left_arm_right_outer_finger, child left_arm_right_inner_finger, origin xyz=0 0.0061 0.0471 rpy=0 0 0, axis 1 0 0, limit lower=-0.8757 upper=0.8757 effort=1000 velocity=2.0, mimic joint=left_arm_finger_joint multiplier=-1 offset=0
- added joint left_arm_right_inner_finger_pad_joint: type fixed, parent left_arm_right_inner_finger, child left_arm_right_inner_finger_pad, origin xyz=0 -0.0220203446692936 0.03242 rpy=0 0 0, axis 0 0 1
- added joint left_arm_right_inner_knuckle_joint: type revolute, parent left_arm_robotiq_arg2f_base_link, child left_arm_right_inner_knuckle, origin xyz=0 0.0127 0.06142 rpy=0 0 0.0, axis 1 0 0, limit lower=0 upper=0.8757 effort=1000 velocity=2.0, mimic joint=left_arm_finger_joint multiplier=1 offset=0
- added joint left_arm_right_outer_finger_joint: type fixed, parent left_arm_right_outer_knuckle, child left_arm_right_outer_finger, origin xyz=0 0.0315 -0.0041 rpy=0 0 0, axis 1 0 0
- added joint left_arm_right_outer_knuckle_joint: type revolute, parent left_arm_robotiq_arg2f_base_link, child left_arm_right_outer_knuckle, origin xyz=0 0.0306011 0.054904 rpy=0 0 0, axis 1 0 0, limit lower=0 upper=0.81 effort=1000 velocity=2.0, mimic joint=left_arm_finger_joint multiplier=1 offset=0
- added joint right_arm_finger_joint: type revolute, parent right_arm_robotiq_arg2f_base_link, child right_arm_left_outer_knuckle, origin xyz=0 -0.0306011 0.054904 rpy=0 0 3.141592653589793, axis 1 0 0, limit lower=0 upper=0.8 effort=1000 velocity=2.0
- added joint right_arm_gripper_base_joint: type fixed, parent right_arm_end_effector_link, child right_arm_robotiq_arg2f_base_link, origin xyz=0.0 0.0 0.0 rpy=0.0 0.0 1.57
- added joint right_arm_left_inner_finger_joint: type revolute, parent right_arm_left_outer_finger, child right_arm_left_inner_finger, origin xyz=0 0.0061 0.0471 rpy=0 0 0, axis 1 0 0, limit lower=-0.8757 upper=0.8757 effort=1000 velocity=2.0, mimic joint=right_arm_finger_joint multiplier=-1 offset=0
- added joint right_arm_left_inner_finger_pad_joint: type fixed, parent right_arm_left_inner_finger, child right_arm_left_inner_finger_pad, origin xyz=0 -0.0220203446692936 0.03242 rpy=0 0 0, axis 0 0 1
- added joint right_arm_left_inner_knuckle_joint: type revolute, parent right_arm_robotiq_arg2f_base_link, child right_arm_left_inner_knuckle, origin xyz=0 -0.0127 0.06142 rpy=0 0 3.141592653589793, axis 1 0 0, limit lower=0 upper=0.8757 effort=1000 velocity=2.0, mimic joint=right_arm_finger_joint multiplier=1 offset=0
- added joint right_arm_left_outer_finger_joint: type fixed, parent right_arm_left_outer_knuckle, child right_arm_left_outer_finger, origin xyz=0 0.0315 -0.0041 rpy=0 0 0, axis 1 0 0
- added joint right_arm_right_inner_finger_joint: type revolute, parent right_arm_right_outer_finger, child right_arm_right_inner_finger, origin xyz=0 0.0061 0.0471 rpy=0 0 0, axis 1 0 0, limit lower=-0.8757 upper=0.8757 effort=1000 velocity=2.0, mimic joint=right_arm_finger_joint multiplier=-1 offset=0
- added joint right_arm_right_inner_finger_pad_joint: type fixed, parent right_arm_right_inner_finger, child right_arm_right_inner_finger_pad, origin xyz=0 -0.0220203446692936 0.03242 rpy=0 0 0, axis 0 0 1
- added joint right_arm_right_inner_knuckle_joint: type revolute, parent right_arm_robotiq_arg2f_base_link, child right_arm_right_inner_knuckle, origin xyz=0 0.0127 0.06142 rpy=0 0 0.0, axis 1 0 0, limit lower=0 upper=0.8757 effort=1000 velocity=2.0, mimic joint=right_arm_finger_joint multiplier=1 offset=0
- added joint right_arm_right_outer_finger_joint: type fixed, parent right_arm_right_outer_knuckle, child right_arm_right_outer_finger, origin xyz=0 0.0315 -0.0041 rpy=0 0 0, axis 1 0 0
- added joint right_arm_right_outer_knuckle_joint: type revolute, parent right_arm_robotiq_arg2f_base_link, child right_arm_right_outer_knuckle, origin xyz=0 0.0306011 0.054904 rpy=0 0 0, axis 1 0 0, limit lower=0 upper=0.81 effort=1000 velocity=2.0, mimic joint=right_arm_finger_joint multiplier=1 offset=0
